Commit message: resolvido problema urdf no rviz

File: src/robot_description/urdf/robot.urdf (robot description, URDF)
Before this commit: robot dinamos_robot, 16 links, 15 joints
Links:
- removed link antebraco_direito
- removed link antebraco_esquerdo
- removed link cotovelo_direito
- removed link cotovelo_esquerdo
- removed link esfera_mao_direito
- removed link esfera_mao_esquerdo
- removed link sensor_camera
- removed link sensor_lidar
- link base_footprint: geometry 
Joints:
- removed joint antebraco_para_mao_direito
- removed joint antebraco_para_mao_esquerdo
- removed joint base_link_para_coluna
- removed joint coluna_para_torso
- removed joint cotovelo_para_antebraco_direito
- removed joint cotovelo_para_antebraco_esquerdo
- removed joint esfera_para_ombro_esquerdo
- removed joint ombro_para_cotovelo_direito
- removed joint ombro_para_cotovelo_esquerdo
- removed joint sensor_camera_torso
- removed joint sensor_lidar_base_link
- removed joint torso_para_esfera_ombro
- removed joint torso_para_esfera_ombro_direito
- added joint base_link_to_coluna: type fixed, parent base_link, child coluna, origin xyz=0 0 0.05 rpy=0 0 0
- added joint coluna_to_torso: type fixed, parent coluna, child torso, origin xyz=0.0 0 0.7 rpy=0 0 0
- added joint esfera_to_ombro_esquerdo: type fixed, parent esfera_ombro_esquerdo, child ombro_esquerdo, origin xyz=0.0 0.0 0.0 rpy=3.14 0 0, axis 1 0 0
- added joint torso_to_esfera_ombro: type fixed, parent torso, child esfera_ombro_esquerdo, origin xyz=0.0 0.085 0.0 rpy=0 0 0
- added joint torso_to_esfera_ombro_direito: type fixed, parent torso, child esfera_ombro_direito, origin xyz=0.0 -0.085 0.0 rpy=0 0 0
- joint base_link_joint: origin xyz=0.0 0 0.0 rpy=0 0 0 -> xyz=0 0 0 rpy=0 0 0
- joint esfera_para_ombro_direito: limit lower=0.0 upper=3.0 effort=30 velocity=0.5 -> (none); type revolute -> fixed

Commit message: adicionado urdf

File: src/robot_description/urdf/robot.urdf (robot description, URDF)
Before this commit: robot robot, 8 links, 7 joints
Links:
- added link antebraco_direito, mass 0.3; collision cylinder length=0.25 radius=0.01; visual cylinder length=0.25 radius=0.01
- added link antebraco_esquerdo, mass 0.3; collision cylinder length=0.25 radius=0.01; visual cylinder length=0.25 radius=0.01
- added link cotovelo_direito, mass 0.15; collision sphere radius=0.02; visual sphere radius=0.02
- added link cotovelo_esquerdo, mass 0.15; collision sphere radius=0.02; visual sphere radius=0.02
- added link esfera_mao_direito, mass 0.05; collision sphere radius=0.02; visual sphere radius=0.02
- added link esfera_mao_esquerdo, mass 0.05; collision sphere radius=0.02; visual sphere radius=0.02
- added link sensor_camera, mass 0.1; collision sphere radius=0.02; visual sphere radius=0.02
- added link sensor_lidar, mass 0.1; collision sphere radius=0.02; visual sphere radius=0.02
Joints:
- added joint antebraco_para_mao_direito: type fixed, parent antebraco_direito, child esfera_mao_direito, origin xyz=0 0 -0.25 rpy=0 0 0, axis 0 1 0
- added joint antebraco_para_mao_esquerdo: type fixed, parent antebraco_esquerdo, child esfera_mao_esquerdo, origin xyz=0 0 -0.25 rpy=0 0 0, axis 0 1 0
- added joint cotovelo_para_antebraco_direito: type fixed, parent cotovelo_direito, child antebraco_direito, origin xyz=0 0 0 rpy=0 0 0, axis 0 1 0
- added joint cotovelo_para_antebraco_esquerdo: type fixed, parent cotovelo_esquerdo, child antebraco_esquerdo, origin xyz=0 0 0 rpy=0 0 0, axis 0 1 0
- added joint ombro_para_cotovelo_direito: type fixed, parent ombro_direito, child cotovelo_direito, origin xyz=0 0 0.20 rpy=3.14 0 0, axis 0 1 0
- added joint ombro_para_cotovelo_esquerdo: type fixed, parent ombro_esquerdo, child cotovelo_esquerdo, origin xyz=0 0 0.20 rpy=3.14 0 0, axis 0 1 0
- added joint sensor_camera_torso: type fixed, parent torso, child sensor_camera, origin xyz=0.075 0.0 0.0 rpy=0 0 0, axis 0 1 0
- added joint sensor_lidar_base_link: type fixed, parent base_link, child sensor_lidar, origin xyz=0.125 0.0 0.05 rpy=0 0 0, axis 0 1 0
